Commit message: updates to urdf/srdf, bugfix joint_1_6achs

File: rod_gruppe9/urdf/combined.urdf (robot description, URDF)
Before this commit: robot combined_robot, 22 links, 21 joints
Joints:
- joint joint_1_6achs: type revolute -> continuous
- joint joint_3_6achs: limit lower=0 upper=3.142 effort=200 velocity=3 -> lower=-1 upper=3.842 effort=200 velocity=3
- joint joint_4: limit lower=-1.57 upper=1.57 effort=200 velocity=3 -> lower=-2 upper=2 effort=200 velocity=3
- joint joint_4_6achs: type revolute -> continuous
- joint joint_5: type revolute -> continuous
- joint joint_6_6achs: type revolute -> continuous

Commit message: positioning of robots and correction to bauteil

File: rod_gruppe9/urdf/combined.urdf (robot description, URDF)
Before this commit: robot combined_robot, 22 links, 21 joints
Joints:
- joint base_joint: origin xyz=0 0 0 rpy=0 0 0 -> xyz=-0.3 0.3 0 rpy=0 0 0
- joint base_joint_6achs: origin xyz=1 1 0 rpy=0 0 0 -> xyz=0.2 0.3 0 rpy=0 0 0
- joint base_joint_stand: origin xyz=2 0 0 rpy=0 0 0 -> xyz=0 -0.4 0 rpy=0 0 0

Commit message: rollback link_6a just gripper, joint standford

File: rod_gruppe9/urdf/combined.urdf (robot description, URDF)
Before this commit: robot combined_robot, 22 links, 21 joints
Joints:
- joint base_joint_stand: origin xyz=0 -0.4 0 rpy=0 0 0 -> xyz=-0.09 -0.35 0 rpy=0 0 -1.5707964
