Commit message: seperation greifen and non greifen

File: rod_gruppe9/urdf/combined_greifen.urdf (robot description, URDF)
Before this commit: robot combined_robot, 25 links, 24 joints
Links:
- removed link bauteil
- removed link bauteil_finished
- removed link bauteil_finished2
Joints:
- removed joint bauteil_finished2_joint
- removed joint bauteil_finished_joint
- removed joint bauteil_joint
